Commit message: 更新URDF和MJCF的轮子碰撞体

File: MujocoSim/scr/atwl/model/at_wheel_leg.urdf (robot description, URDF)
Before this commit: robot at_wheel_leg, 15 links, 14 joints
Links:
- link left_wheel_link: geometry collision cylinder length=0.021 radius=0.056; visual mesh filename=left_wheel_link.STL
- link right_wheel_link: geometry collision cylinder length=0.021 radius=0.056; visual mesh filename=right_wheel_link.STL

Commit message: 修正URDF和MJCF文件的错误

File: MujocoSim/scr/atwl/model/at_wheel_leg.urdf (robot description, URDF)
Before this commit: robot at_wheel_leg, 15 links, 14 joints
Joints:
- joint right_rear2_link_right_wheel_link_joint: axis 0 -1 0 -> 0 1 0
